Commit message: Trim GMR into a G1/H1 offline-retargeting fork (COLMO)
- Keep only Unitree G1 and H1; remove the other ~18 robots (assets, params,
  IK configs, and script --robot choices).
- Remove real-time teleoperation: OptiTrack (optitrack_to_robot + optitrack_vendor)
  and XR/PICO (xrobot_utils); drop the "fbx"/"xrobot" input sources.
- Remove the scale/offset calibration feature (calibrate_offsets_from_initial_pose,
  vis_calibrate_scale.py, --scale_mode calib) and neck_retarget.py; drop dead code.
- Collision avoidance: soft barrier removed; modes are now cbf/issf/off (default
  issf). Add a soft per-frame acceleration limit (DAQP sense=8).
- Externalize hardcoded IK params to collision_cfg.yaml (solver, warmup_iters,
  ik_convergence_tol, lm_damping, motion_fps, ground_offset/ground_lift); make
  damping/max_iter/velocity_limit required.
- Add README.md for scripts/ and general_motion_retargeting/; clean up main README.
- gitignore amass/.

Co-Authored-By: Claude Opus 4.8 <noreply@anthropic.com>

File: assets/unitree_g1/g1_custom_collision_29dof.urdf (robot description, URDF)
Before this commit: robot g1_29dof_rev_1_0, 38 links, 37 joints
Joints:
- joint left_shoulder_pitch_joint: limit lower=-3.0892 upper=2.6704 effort=25 velocity=37 -> lower=-3.0892 upper=1.649 effort=25 velocity=37
- joint right_shoulder_pitch_joint: limit lower=-3.0892 upper=2.6704 effort=25 velocity=37 -> lower=-3.0892 upper=1.649 effort=25 velocity=37
