Commit message: delte shoulder yaw tracking

File: assets/unitree_g1/g1_custom_collision_29dof.urdf (robot description, URDF)
Before this commit: robot g1_29dof_rev_1_0, 38 links, 37 joints
Joints:
- joint left_shoulder_pitch_joint: limit lower=-3.0892 upper=1.649 effort=25 velocity=37 -> lower=-2.6 upper=0.95 effort=25 velocity=37
- joint right_shoulder_pitch_joint: limit lower=-3.0892 upper=1.649 effort=25 velocity=37 -> lower=-2.6 upper=0.95 effort=25 velocity=37
